Commit message: sim nav working, bad urdf tho

File: src/zbig_description/urdf/bigbot_gazebo_control.xacro (robot description, xacro)
@@ -98,5 +98,5 @@
    <!-- 2D Laser Sensor -->
    <gazebo reference="laser_frame">
-    <sensor name="lidar" type="gpu_lidar">
+    <sensor name="gpu_lidar" type="gpu_lidar">
       <always_on>true</always_on>
       <visualize>true</visualize>
@@ -109,6 +109,6 @@
             <samples>360</samples>
             <resolution>1.00000</resolution>
-            <min_angle>0.000000</min_angle>
-            <max_angle>6.280000</max_angle>
+            <min_angle>-3.1416</min_angle>
+            <max_angle>3.1416</max_angle>
           </horizontal>
         </scan>
@@ -195,3 +195,14 @@
   </gazebo>
   -->
+  <gazebo reference="base_link">
+    <sensor name="navsat" type="navsat">
+      <always_on>1</always_on>
+      <!--  -->
+      <update_rate>1</update_rate>
+      <!---->
+      <topic>navsat</topic>
+      <!---->
+      <gz_frame_id>base_link</gz_frame_id>
+    </sensor>
+  </gazebo>
 </robot>

File: src/zbig_description/urdf/bigbot_physical.urdf.xacro (robot description, xacro)
@@ -39,5 +39,5 @@
     <parent link="base_footprint"/>
     <child link="base_link" />
-    <origin xyz="0 0 0.063" rpy="0 0 0"/>
+    <origin xyz="0 0 0.074" rpy="0 0 0"/>
   </joint>
   <link name="wheel_right_link">
@@ -177,5 +177,5 @@
   </link>
   <joint name="imu_joint" type="fixed">
-    <origin xyz="-0.04016 0.049755 0.064953" rpy="3.14 0 -1.57" />
+    <origin xyz="-0.04016 0.049755 0.064953" rpy="0 0 1.57" />
     <parent link="base_link" />
     <child link="imu_link" />
@@ -205,5 +205,5 @@
   </link>
   <joint name="laser_joint" type="fixed">
-    <origin xyz="-0.013456 0.000513 0.140452" rpy="0 0 3.14" />
+    <origin xyz="-0.013456 0.000513 0.140452" rpy="0 0 0" />
     <parent link="base_link" />
     <child link="laser_frame" />

Commit message: corrected lidar fov

File: src/zbig_description/urdf/bigbot_gazebo_control.xacro (robot description, xacro)
@@ -109,6 +109,6 @@
             <samples>360</samples>
             <resolution>1.00000</resolution>
-            <min_angle>0.0</min_angle>
-            <max_angle>6.28</max_angle>
+            <min_angle>-2.269</min_angle>
+            <max_angle>2.269</max_angle>
           </horizontal>
         </scan>

File: src/zbig_description/urdf/bigbot_physical.urdf.xacro (robot description, xacro)
@@ -10,8 +10,8 @@
     <xacro:property name="imu_roll" value="0.0"/>
     <xacro:property name="imu_pitch" value="0.0"/>
-    <xacro:property name="imu_yaw" value="0.0"/>
+    <xacro:property name="imu_yaw" value="3.14"/>
     <xacro:property name="lidar_roll" value="0.0"/>
     <xacro:property name="lidar_pitch" value="0.0"/>
-    <xacro:property name="lidar_yaw" value="3.14"/>
+    <xacro:property name="lidar_yaw" value="0.0"/>
     <xacro:property name="chassis_mass" value="10.0"/>
     <xacro:property name="wheel_mass" value="0.05"/>
@@ -196,5 +196,5 @@
   <link name="laser_frame">
     <inertial>
-      <origin xyz="0.005399 -0.010876 0.002517" rpy="0 0 0" />
+      <origin xyz="0.005399 -0.010876 0.002517" rpy="0 0 ${lidar_yaw}" />
       <mass value="0.07308" />
       <inertia ixx="0.000039" ixy="-0.000011" ixz="0.000003"

Commit message: lidar orientation change

File: src/zbig_description/urdf/bigbot_gazebo_control.xacro (robot description, xacro)
@@ -109,6 +109,6 @@
             <samples>360</samples>
             <resolution>1.00000</resolution>
-            <min_angle>-2.269</min_angle>
-            <max_angle>2.269</max_angle>
+            <min_angle>0</min_angle>
+            <max_angle>6.28</max_angle>
           </horizontal>
         </scan>

File: src/zbig_description/urdf/bigbot_physical.urdf.xacro (robot description, xacro)
@@ -208,5 +208,5 @@
     </inertial>
     <visual>
-      <origin xyz="0 0 0" rpy="1.57 0 3.14" />
+      <origin xyz="0 0 0" rpy="1.57 0 0" />
       <geometry>
         <mesh filename="file://$(find zbig_description)/meshes/lidarA1M8.stl" />

Commit message: narrowbot1 initial upload

File: src/zbig_description/urdf/bigbot_gazebo_control.xacro (robot description, xacro)
@@ -109,6 +109,6 @@
             <samples>360</samples>
             <resolution>1.00000</resolution>
-            <min_angle>0</min_angle>
-            <max_angle>6.28</max_angle>
+            <min_angle>-2.3</min_angle>
+            <max_angle>2.3</max_angle>
           </horizontal>
         </scan>

File: src/zbig_description/urdf/bigbot_physical.urdf.xacro (robot description, xacro)
@@ -14,8 +14,8 @@
     <xacro:property name="lidar_pitch" value="0.0"/>
     <xacro:if value="$(arg is_sim)">
-      <xacro:property name="lidar_yaw" value="3.14"/>
+      <xacro:property name="lidar_yaw" value="0.0"/>
     </xacro:if>
     <xacro:unless value="$(arg is_sim)">
-      <xacro:property name="lidar_yaw" value="3.14"/>
+      <xacro:property name="lidar_yaw" value="0.0"/>
     </xacro:unless>
     <xacro:property name="chassis_mass" value="10.0"/>
@@ -36,5 +36,5 @@
       <origin xyz="0 0 0" rpy="0 0 0" />
       <geometry>
-        <mesh filename="file://$(find zbig_description)/meshes/smallbot_base_link.stl" />
+        <mesh filename="file://$(find zbig_description)/meshes/narrowbot/collision-chassis-narrow1.stl" />
       </geometry>
       <material name="dark_grey"/>
@@ -43,5 +43,5 @@
       <origin xyz="0 0 0" rpy="0 0 0" />
       <geometry>
-        <mesh filename="file://$(find zbig_description)/meshes/smallbot_base_link.stl" />
+        <mesh filename="file://$(find zbig_description)/meshes/narrowbot/collision-chassis-narrow1.stl" />
       </geometry>
     </collision>
@@ -64,5 +64,5 @@
       <origin xyz="-0.0 0.014 0.0" rpy="1.57 0 0" />
       <geometry>
-        <mesh filename="file://$(find zbig_description)/meshes/smallbot_wheel.stl" />
+        <mesh filename="file://$(find zbig_description)/meshes/narrowbot/collision-6inch-wheel.stl" />
       </geometry>
       <material name="blue"/>
@@ -94,5 +94,5 @@
       <origin xyz="0 -0.014 0" rpy="-1.57 0 0" />
       <geometry>
-        <mesh filename="file://$(find zbig_description)/meshes/smallbot_wheel.stl" />
+        <mesh filename="file://$(find zbig_description)/meshes/narrowbot/collision-6inch-wheel.stl" />
       </geometry>
       <material name="blue"/>
@@ -121,7 +121,7 @@
     </inertial>
     <visual>
-      <origin xyz="0 0 0" rpy="0 0 0" />
-      <geometry>
-        <mesh filename="file://$(find zbig_description)/meshes/smallbot_caster_link.stl" />
+      <origin xyz="0 ${wheel_offset_z} 0" rpy="0 0 0" />
+      <geometry>
+        <mesh filename="file://$(find zbig_description)/meshes/narrowbot/visual-caster-narrow1.stl" />
       </geometry>
       <material name="silver"/>
@@ -150,7 +150,7 @@
     </inertial>
     <visual>
-      <origin xyz="0 0 0" rpy="0 0 0" />
-      <geometry>
-        <mesh filename="file://$(find zbig_description)/meshes/smallbot_caster_link.stl" />
+      <origin xyz="0 ${wheel_offset_z} 0" rpy="0 0 0" />
+      <geometry>
+         <mesh filename="file://$(find zbig_description)/meshes/narrowbot/visual-caster-narrow1.stl" />
       </geometry>
       <material name="silver"/>
@@ -179,19 +179,19 @@
     </inertial>
     <visual>
-      <origin xyz="0 0 0" rpy="0 0 0" />
-      <geometry>
-        <mesh filename="file://$(find zbig_description)/meshes/imu_link.STL" />
+      <origin xyz="0.1 0 -.10" rpy="0 0 0" />
+      <geometry>
+        <mesh filename="file://$(find zbig_description)/meshes/narrowbot/collision-imu.stl" />
       </geometry>
       <material name="blue"/>
     </visual>
     <collision>
-      <origin xyz="0 0 0" rpy="${imu_roll} ${imu_pitch} ${imu_yaw}" />
-      <geometry>
-        <mesh filename="file://$(find zbig_description)/meshes/imu_link.STL" />
+      <origin xyz="0.1 0 -.10" rpy="${imu_roll} ${imu_pitch} ${imu_yaw}" />
+      <geometry>
+        <mesh filename="file://$(find zbig_description)/meshes/narrowbot/collision-imu.stl" />
       </geometry>
     </collision>
   </link>
   <joint name="imu_joint" type="fixed">
-    <origin xyz="-0.04016 0.049755 0.064953" rpy="${imu_roll} ${imu_pitch} ${imu_yaw}" />
+    <origin xyz="-0.04016 0.049755 0.1" rpy="${imu_roll} ${imu_pitch} ${imu_yaw}" />
     <parent link="base_link" />
     <child link="imu_link" />
@@ -210,5 +210,5 @@
       <origin xyz="0 0 0" rpy="1.57 0 0" />
       <geometry>
-        <mesh filename="file://$(find zbig_description)/meshes/lidarA1M8.stl" />
+        <mesh filename="file://$(find zbig_description)/meshes/narrowbot/collision-lidar.stl" />
       </geometry>
       <material name="black"/>
@@ -217,5 +217,5 @@
       <origin xyz="0 0 0" rpy="${lidar_roll} ${lidar_pitch} ${lidar_yaw}" />
       <geometry>
-        <mesh filename="file://$(find zbig_description)/meshes/lidarA1M8.stl" />
+        <mesh filename="file://$(find zbig_description)/meshes/narrowbot/collision-lidar.stl" />
       </geometry>
     </collision>

Commit message: corrected bigbot dimensions

File: src/zbig_description/urdf/bigbot_gazebo_control.xacro (robot description, xacro)
@@ -109,6 +109,6 @@
             <samples>360</samples>
             <resolution>1.00000</resolution>
-            <min_angle>-2.3</min_angle>
-            <max_angle>2.3</max_angle>
+            <min_angle>0</min_angle>
+            <max_angle>6.28</max_angle>
           </horizontal>
         </scan>

File: src/zbig_description/urdf/bigbot_physical.urdf.xacro (robot description, xacro)
@@ -2,9 +2,9 @@
 <robot name="zbig" xmlns:xacro="http://ros.org/wiki/xacro">
     <xacro:property name="wheel_radius" value="0.074"/>
-    <xacro:property name="wheel_offset_y" value="0.2225"/>
+    <xacro:property name="wheel_offset_y" value="0.235"/>
     <xacro:property name="wheel_offset_z" value="0.0225"/>
     <xacro:property name="caster_wheel_radius" value="0.051"/>
-    <xacro:property name="caster_wheel_offset_x" value="0.137"/>
-    <xacro:property name="caster_wheel_offset_y" value="0.095"/>
+    <xacro:property name="caster_wheel_offset_x" value="0.280"/>
+    <xacro:property name="caster_wheel_offset_y" value="0.138"/>
     <xacro:property name="caster_wheel_offset_z" value="${wheel_offset_z - wheel_radius + caster_wheel_radius}"/>
     <xacro:property name="imu_roll" value="0.0"/>
@@ -36,5 +36,5 @@
       <origin xyz="0 0 0" rpy="0 0 0" />
       <geometry>
-        <mesh filename="file://$(find zbig_description)/meshes/narrowbot/collision-chassis-narrow1.stl" />
+        <mesh filename="file://$(find zbig_description)/meshes/collision-chassis-bigbot1.stl" />
       </geometry>
       <material name="dark_grey"/>
@@ -43,5 +43,5 @@
       <origin xyz="0 0 0" rpy="0 0 0" />
       <geometry>
-        <mesh filename="file://$(find zbig_description)/meshes/narrowbot/collision-chassis-narrow1.stl" />
+        <mesh filename="file://$(find zbig_description)/meshes/collision-chassis-bigbot1.stl" />
       </geometry>
     </collision>
@@ -55,5 +55,5 @@
   <link name="wheel_right_link">
     <inertial>
-      <origin xyz="0 -0.014 0" rpy="0 0 0" />
+      <origin xyz="0 0.0 0" rpy="0 0 0" />
       <mass value="${wheel_mass}" />
       <inertia ixx="1.88176298336665E-05" ixy="-4.8444933029987E-10" ixz="1.88163708851143E-08"
@@ -62,5 +62,5 @@
     </inertial>
     <visual>
-      <origin xyz="-0.0 0.014 0.0" rpy="1.57 0 0" />
+      <origin xyz="-0.0 0.0 0.0" rpy="1.57 0 0" />
       <geometry>
         <mesh filename="file://$(find zbig_description)/meshes/narrowbot/collision-6inch-wheel.stl" />
@@ -85,5 +85,5 @@
     name="wheel_left_link">
     <inertial>
-      <origin xyz="0 -0.014 0" rpy="0 0 0" />
+      <origin xyz="0 0.0 0" rpy="0 0 0" />
       <mass value="${wheel_mass}" />
       <inertia ixx="1.8792911368909E-05"  ixy="3.31256392204584E-10" ixz="-1.14082001662767E-08"
@@ -92,5 +92,5 @@
     </inertial>
     <visual>
-      <origin xyz="0 -0.014 0" rpy="-1.57 0 0" />
+      <origin xyz="0 0.0 0" rpy="-1.57 0 0" />
       <geometry>
         <mesh filename="file://$(find zbig_description)/meshes/narrowbot/collision-6inch-wheel.stl" />
@@ -121,5 +121,5 @@
     </inertial>
     <visual>
-      <origin xyz="0 ${wheel_offset_z} 0" rpy="0 0 0" />
+      <origin xyz="0 ${wheel_offset_z} 0" rpy="0 1.57 0" />
       <geometry>
         <mesh filename="file://$(find zbig_description)/meshes/narrowbot/visual-caster-narrow1.stl" />
@@ -150,5 +150,5 @@
     </inertial>
     <visual>
-      <origin xyz="0 ${wheel_offset_z} 0" rpy="0 0 0" />
+      <origin xyz="0 ${wheel_offset_z} 0" rpy="0 -1.57 0.0" />
       <geometry>
          <mesh filename="file://$(find zbig_description)/meshes/narrowbot/visual-caster-narrow1.stl" />
@@ -193,5 +193,5 @@
   </link>
   <joint name="imu_joint" type="fixed">
-    <origin xyz="-0.04016 0.049755 0.1" rpy="${imu_roll} ${imu_pitch} ${imu_yaw}" />
+    <origin xyz="-0.140 0.023 0.31" rpy="${imu_roll} ${imu_pitch} ${imu_yaw}" />
     <parent link="base_link" />
     <child link="imu_link" />
@@ -222,5 +222,5 @@
   </link>
   <joint name="laser_joint" type="fixed">
-    <origin xyz="-0.013456 0.000513 0.140452" rpy="${lidar_roll} ${lidar_pitch} ${lidar_yaw}" />
+    <origin xyz="-0.035 0.000 0.4" rpy="${lidar_roll} ${lidar_pitch} ${lidar_yaw}" />
     <parent link="base_link" />
     <child link="laser_frame" />
