Commit message: sim of nav with slam works

File: src/zbig_description/urdf/bigbot.urdf.xacro (robot description, xacro)
@@ -6,4 +6,5 @@
   <!-- Include physical aspects of the robot, includes LIDAR and IMU -->
   <xacro:include filename="$(find zbig_description)/urdf/bigbot_physical.urdf.xacro" />
+  <xacro:include filename="$(find zbig_description)/urdf/materials.xacro" />
   <!-- Include ros2 control Parameters for both SIM and REAL robots-->
   <xacro:include filename="$(find zbig_description)/urdf/bigbot_ros2_control.xacro" />

File: src/zbig_description/urdf/bigbot_gazebo_control.xacro (robot description, xacro)
@@ -195,14 +195,3 @@
   </gazebo>
   -->
-  <gazebo reference="base_link">
-    <sensor name="navsat" type="navsat">
-      <always_on>1</always_on>
-      <!--  -->
-      <update_rate>1</update_rate>
-      <!---->
-      <topic>navsat</topic>
-      <!---->
-      <gz_frame_id>base_link</gz_frame_id>
-    </sensor>
-  </gazebo>
 </robot>

File: src/zbig_description/urdf/bigbot_physical.urdf.xacro (robot description, xacro)
@@ -1,26 +1,32 @@
 <?xml version="1.0"?>
 <robot name="zbig" xmlns:xacro="http://ros.org/wiki/xacro">
-  <material name="blue">
-    <color rgba="0 0 1 1"/>
-  </material>
-  <material name="black">
-    <color rgba="0 0 0 1"/>
-  </material>
-  <material name="silver">
-    <color rgba="0.79 0.82 0.93 1"/>
-  </material>
-  <material name="dark_grey">
-    <color rgba="0.3 0.3 0.3 1"/>
-  </material>
-  <link name="base_footprint"/>
+    <xacro:property name="wheel_radius" value="0.074"/>
+    <xacro:property name="wheel_offset_y" value="0.2225"/>
+    <xacro:property name="wheel_offset_z" value="0.0225"/>
+    <xacro:property name="caster_wheel_radius" value="0.051"/>
+    <xacro:property name="caster_wheel_offset_x" value="0.137"/>
+    <xacro:property name="caster_wheel_offset_y" value="0.095"/>
+    <xacro:property name="caster_wheel_offset_z" value="${wheel_offset_z - wheel_radius + caster_wheel_radius}"/>
+    <xacro:property name="imu_roll" value="0.0"/>
+    <xacro:property name="imu_pitch" value="0.0"/>
+    <xacro:property name="imu_yaw" value="1.57"/>
+    <xacro:property name="lidar_roll" value="0.0"/>
+    <xacro:property name="lidar_pitch" value="0.0"/>
+    <xacro:property name="lidar_yaw" value="0.0"/>
+    <xacro:property name="chassis_mass" value="10.0"/>
+    <xacro:property name="wheel_mass" value="0.05"/>
+    <xacro:property name="caster_wheel_mass" value="0.01"/>
+  <!-- BASE_FOOTPRINT LINK -->
+  <link name="base_footprint"></link>
+   <!-- BASE LINK -->
   <link name="base_link">
     <inertial>
       <origin xyz="-0.070489 -0.000718 0.040699" rpy="0.0 0.0 0.0" />
-      <mass value="10.0"/>
+      <mass value="${chassis_mass}"/>
       <inertia ixx="0.011114" ixy="0.000188" ixz="-0.005821"
                iyy="0.017229" iyz="0.000127"
                izz="0.019734" />
     </inertial>
-    <visual>
+    <visual name='base_link_visual'>
       <origin xyz="0 0 0" rpy="0 0 0" />
       <geometry>
@@ -36,13 +42,14 @@
     </collision>
   </link>
-  <joint name="base_joint" type="fixed">
+   <joint name="base_joint" type="fixed">
     <parent link="base_footprint"/>
     <child link="base_link" />
-    <origin xyz="0 0 0.074" rpy="0 0 0"/>
-  </joint>
+    <origin xyz="0 0 ${wheel_radius}" rpy="0 0 0"/>
+  </joint>
+<!-- RIGHT WHEEL LINK -->
   <link name="wheel_right_link">
     <inertial>
       <origin xyz="0 -0.014 0" rpy="0 0 0" />
-      <mass value="0.0530086090966721" />
+      <mass value="${wheel_mass}" />
       <inertia ixx="1.88176298336665E-05" ixy="-4.8444933029987E-10" ixz="1.88163708851143E-08"
                iyy="3.11510738647764E-05" iyz="-6.93560663069607E-11"
@@ -59,19 +66,20 @@
       <origin xyz="0 -0.015 0" rpy="1.57 0 0" />
       <geometry>
-        <sphere radius="0.063"/>
+        <sphere radius="${wheel_radius}"/>
       </geometry>
     </collision>
   </link>
   <joint name="wheel_right_joint" type="continuous">
-    <origin xyz="0 -0.2225 0" rpy="0 0 0" />
+    <origin xyz="0 ${-wheel_offset_y} 0" rpy="0 0 0" />
     <parent link="base_link" />
     <child link="wheel_right_link" />
     <axis xyz="0 1 0" />
   </joint>
+<!-- LEFT WHEEL LINK -->
   <link
     name="wheel_left_link">
     <inertial>
       <origin xyz="0 -0.014 0" rpy="0 0 0" />
-      <mass value="0.0530086043217644" />
+      <mass value="${wheel_mass}" />
       <inertia ixx="1.8792911368909E-05"  ixy="3.31256392204584E-10" ixz="-1.14082001662767E-08"
                iyy="3.11510738759073E-05" iyz="-3.60499245082192E-10"
@@ -88,14 +96,15 @@
       <origin xyz="0 -0.014 0" rpy="-1.57 0 0" />
       <geometry>
-        <sphere radius="0.063"/>
+        <sphere radius="${wheel_radius}"/>
       </geometry>
     </collision>
   </link>
   <joint name="wheel_left_joint" type="continuous">
-    <origin xyz="0 0.2225 0" rpy="0 0 0" />
+    <origin xyz="0 ${wheel_offset_y}  0" rpy="0 0 0" />
     <parent link="base_link" />
     <child link="wheel_left_link" />
     <axis xyz="0 1 0" />
   </joint>
+<!-- RIGHT CASTER WHEEL LINK -->
   <link name="caster_right_link">
     <inertial>
@@ -116,14 +125,15 @@
       <origin xyz="0 0 0" rpy="0 0 0" />
       <geometry>
-        <sphere radius="0.051"/>
+        <sphere radius="${wheel_radius}"/>
       </geometry>
     </collision>
   </link>
   <joint name="caster_right_joint" type="fixed">
-    <origin xyz="-0.137 -0.095 -.025" rpy="1.57 0 1.57" />
+    <origin xyz="${-caster_wheel_offset_x} ${-caster_wheel_offset_y} ${-caster_wheel_offset_z}" rpy="1.57 0 1.57" />
     <parent link="base_link" />
     <child link="caster_right_link" />
     <axis xyz="0 0 0" />
   </joint>
+<!-- LEFT CASTER WHEEL LINK -->
   <link name="caster_left_link">
     <inertial>
@@ -144,14 +154,15 @@
       <origin xyz="0 0 0" rpy="0 0 0" />
       <geometry>
-        <sphere radius="0.051"/>
+        <sphere radius="${wheel_radius}"/>
       </geometry>
     </collision>
   </link>
   <joint name="caster_left_joint" type="fixed">
-    <origin xyz="-0.137 0.095 -.025" rpy="1.57 0 1.57" />
+    <origin xyz="${-caster_wheel_offset_x} ${caster_wheel_offset_y} ${-caster_wheel_offset_z}" rpy="1.57 0 1.57" />
     <parent link="base_link" />
     <child link="caster_left_link" />
     <axis xyz="0 0 0" />
   </joint>
+<!-- IMU LINK -->
   <link name="imu_link">
     <inertial>
@@ -170,5 +181,5 @@
     </visual>
     <collision>
-      <origin xyz="0 0 0" rpy="0 0 1.57" />
+      <origin xyz="0 0 0" rpy="${imu_roll} ${imu_pitch} ${imu_yaw}" />
       <geometry>
         <mesh filename="file://$(find zbig_description)/meshes/imu_link.STL" />
@@ -177,9 +188,10 @@
   </link>
   <joint name="imu_joint" type="fixed">
-    <origin xyz="-0.04016 0.049755 0.064953" rpy="0 0 1.57" />
+    <origin xyz="-0.04016 0.049755 0.064953" rpy="${imu_roll} ${imu_pitch} ${imu_yaw}" />
     <parent link="base_link" />
     <child link="imu_link" />
     <axis xyz="0 0 0" />
   </joint>
+<!-- LIDAR LINK -->
   <link name="laser_frame">
     <inertial>
@@ -198,5 +210,5 @@
     </visual>
     <collision>
-      <origin xyz="0 0 0" rpy="0 0 0" />
+      <origin xyz="0 0 0" rpy="${lidar_roll} ${lidar_pitch} ${lidar_yaw}" />
       <geometry>
         <mesh filename="file://$(find zbig_description)/meshes/lidarA1M8.stl" />
@@ -205,5 +217,5 @@
   </link>
   <joint name="laser_joint" type="fixed">
-    <origin xyz="-0.013456 0.000513 0.140452" rpy="0 0 0" />
+    <origin xyz="-0.013456 0.000513 0.140452" rpy="${lidar_roll} ${lidar_pitch} ${lidar_yaw}" />
     <parent link="base_link" />
     <child link="laser_frame" />

Commit message: depth nav simulation initial try

File: src/zbig_description/urdf/bigbot.urdf.xacro (robot description, xacro)
@@ -14,5 +14,5 @@
   </xacro:if>
   <!-- Include sensors -->
-  <!-- <xacro:include filename="$(find zbig_description)/urdf/camera.xacro" /> -->
+  <xacro:include filename="$(find zbig_description)/urdf/camera.xacro" />
   <xacro:include filename="$(find zbig_description)/urdf/depth_camera.xacro" />
 </robot>

File: src/zbig_description/urdf/depth_camera.xacro (robot description, xacro)
@@ -1,41 +1,57 @@
 <?xml version="1.0"?>
 <robot xmlns:xacro="http://www.ros.org/wiki/xacro" >
-    <joint name="camera_joint" type="fixed">
+    <joint name="depth_camera_joint" type="fixed">
         <parent link="base_link"/>
-        <child link="camera_link"/>
-        <origin xyz="0.08 0 0.300" rpy="0 0 0"/>
+        <child link="depth_camera_link"/>
+        <origin xyz="0.08 0.0 0.350" rpy="0 0 0"/>
     </joint>
-    <link name="camera_link">
+    <link name="depth_camera_link">
         <visual>
             <geometry>
                 <box size="0.010 0.03 0.03"/>
             </geometry>
-            <material name="red"/>
+            <material name="blue"/>
         </visual>
     </link>
-    <joint name="camera_optical_joint" type="fixed">
-        <parent link="camera_link"/>
-        <child link="camera_link_optical"/>
+    <joint name="depth_camera_optical_joint" type="fixed">
+        <parent link="depth_camera_link"/>
+        <child link="depth_camera_link_optical"/>
         <origin xyz="0 0 0" rpy="${-pi/2} 0 ${-pi/2}"/>
     </joint>
-    <link name="camera_link_optical"></link>
-    <gazebo reference="camera_link">
+    <link name="depth_camera_link_optical"></link>
+    <gazebo reference="depth_camera_link">
         <material>Gazebo/Red</material>
-        <sensor name="depth_camera1" type="depth_camera">
-          <update_rate>10</update_rate>
-          <topic>depth_camera</topic>
-          <camera>
-            <horizontal_fov>1.05</horizontal_fov>
-            <image>
-              <width>256</width>
-              <height>256</height>
-              <format>R_FLOAT32</format>
-            </image>
-            <clip>
-              <near>0.1</near>
-              <far>10.0</far>
-            </clip>
-          </camera>
-          </sensor>
+      <sensor name="depth_camera" type="rgbd_camera">
+        <always_on>true</always_on>
+        <visualize>true</visualize>
+        <update_rate>5.0</update_rate>
+        <topic>depth_camera</topic>
+        <gz_frame_id>depth_camera_link</gz_frame_id>
+        <camera>
+          <horizontal_fov>2.3</horizontal_fov>
+          <!-- <vertical_fov>0.5</vertical_fov> -->
+          <image>
+            <width>480</width>
+            <height>480</height>
+          </image>
+          <clip>
+            <near>0.05</near>
+            <far>3</far>
+          </clip>
+        </camera>
+        <baseline>0.2</baseline>
+        <pointCloudCutoff>0.5</pointCloudCutoff>
+        <pointCloudCutoffMax>3.0</pointCloudCutoffMax>
+        <distortionK1>0</distortionK1>
+        <distortionK2>0</distortionK2>
+        <distortionK3>0</distortionK3>
+        <distortionT1>0</distortionT1>
+        <distortionT2>0</distortionT2>
+        <CxPrime>0</CxPrime>
+        <Cx>0</Cx>
+        <Cy>0</Cy>
+        <focalLength>0</focalLength>
+        <hackBaseline>0</hackBaseline>
+      </sensor>
     </gazebo>
 </robot>

File: src/zbig_description/urdf/lidar_narrowbot.xacro (robot description, xacro)
@@ -47,6 +47,6 @@
             <samples>360</samples>
             <resolution>1.00000</resolution>
-            <min_angle>0</min_angle>
-            <max_angle>6.28</max_angle>
+            <min_angle>-2.2</min_angle>
+            <max_angle>2.2</max_angle>
           </horizontal>
         </scan>
