Commit message: lidar orientation reversed

File: src/zbig_description/urdf/bigbot_physical.urdf.xacro (robot description, xacro)
@@ -13,5 +13,5 @@
     <xacro:property name="lidar_roll" value="0.0"/>
     <xacro:property name="lidar_pitch" value="0.0"/>
-    <xacro:property name="lidar_yaw" value="0.0"/>
+    <xacro:property name="lidar_yaw" value="3.14"/>
     <xacro:property name="chassis_mass" value="10.0"/>
     <xacro:property name="wheel_mass" value="0.05"/>

Commit message: enable ekf in both sim and real hw

File: src/zbig_description/urdf/bigbot_physical.urdf.xacro (robot description, xacro)
@@ -64,5 +64,5 @@
     </visual>
     <collision>
-      <origin xyz="0 -0.015 0" rpy="1.57 0 0" />
+      <origin xyz="0 0 0" rpy="1.57 0 0" />
       <geometry>
         <sphere radius="${wheel_radius}"/>
@@ -94,5 +94,5 @@
     </visual>
     <collision>
-      <origin xyz="0 -0.014 0" rpy="-1.57 0 0" />
+      <origin xyz="0 0 0" rpy="-1.57 0 0" />
       <geometry>
         <sphere radius="${wheel_radius}"/>

Commit message: turned imu x toward front

File: src/zbig_description/urdf/bigbot_physical.urdf.xacro (robot description, xacro)
@@ -10,5 +10,5 @@
     <xacro:property name="imu_roll" value="0.0"/>
     <xacro:property name="imu_pitch" value="0.0"/>
-    <xacro:property name="imu_yaw" value="1.57"/>
+    <xacro:property name="imu_yaw" value="0.0"/>
     <xacro:property name="lidar_roll" value="0.0"/>
     <xacro:property name="lidar_pitch" value="0.0"/>
@@ -174,5 +174,5 @@
     </inertial>
     <visual>
-      <origin xyz="0 0 0" rpy="0 0 3.14" />
+      <origin xyz="0 0 0" rpy="0 0 0" />
       <geometry>
         <mesh filename="file://$(find zbig_description)/meshes/imu_link.STL" />

Commit message: corrected imu yaw in urdf

File: src/zbig_description/urdf/bigbot_physical.urdf.xacro (robot description, xacro)
@@ -10,5 +10,5 @@
     <xacro:property name="imu_roll" value="0.0"/>
     <xacro:property name="imu_pitch" value="0.0"/>
-    <xacro:property name="imu_yaw" value="3.14"/>
+    <xacro:property name="imu_yaw" value="0.0"/>
     <xacro:property name="lidar_roll" value="0.0"/>
     <xacro:property name="lidar_pitch" value="0.0"/>

Commit message: made lidar yaw different for sim & real bot

File: src/zbig_description/urdf/bigbot_physical.urdf.xacro (robot description, xacro)
@@ -13,5 +13,10 @@
     <xacro:property name="lidar_roll" value="0.0"/>
     <xacro:property name="lidar_pitch" value="0.0"/>
-    <xacro:property name="lidar_yaw" value="0.0"/>
+    <xacro:if value="$(arg is_sim)">
+      <xacro:property name="lidar_yaw" value="0.00"/>
+    </xacro:if>
+    <xacro:unless value="$(arg is_sim)">
+      <xacro:property name="lidar_yaw" value="3.14"/>
+    </xacro:unless>
     <xacro:property name="chassis_mass" value="10.0"/>
     <xacro:property name="wheel_mass" value="0.05"/>

Commit message: back to navigation.yaml with mppi & shim

File: src/zbig_description/urdf/bigbot_physical.urdf.xacro (robot description, xacro)
@@ -14,5 +14,5 @@
     <xacro:property name="lidar_pitch" value="0.0"/>
     <xacro:if value="$(arg is_sim)">
-      <xacro:property name="lidar_yaw" value="0.00"/>
+      <xacro:property name="lidar_yaw" value="3.14"/>
     </xacro:if>
     <xacro:unless value="$(arg is_sim)">

Commit message: tuning bigbot urdf and nav

File: src/zbig_description/urdf/bigbot_physical.urdf.xacro (robot description, xacro)
@@ -13,10 +13,5 @@
     <xacro:property name="lidar_roll" value="0.0"/>
     <xacro:property name="lidar_pitch" value="0.0"/>
-    <xacro:if value="$(arg is_sim)">
-      <xacro:property name="lidar_yaw" value="0.0"/>
-    </xacro:if>
-    <xacro:unless value="$(arg is_sim)">
-      <xacro:property name="lidar_yaw" value="0.0"/>
-    </xacro:unless>
+    <xacro:property name="lidar_yaw" value="0.0"/>
     <xacro:property name="chassis_mass" value="10.0"/>
     <xacro:property name="wheel_mass" value="0.05"/>
@@ -29,7 +24,7 @@
       <origin xyz="-0.070489 -0.000718 0.040699" rpy="0.0 0.0 0.0" />
       <mass value="${chassis_mass}"/>
-      <inertia ixx="0.011114" ixy="0.000188" ixz="-0.005821"
-               iyy="0.017229" iyz="0.000127"
-               izz="0.019734" />
+      <inertia ixx="0.4947" ixy="0.00" ixz="-0.1925"
+               iyy="0.6072" iyz="0.00"
+               izz="0.4081" />
     </inertial>
     <visual name='base_link_visual'>
@@ -179,5 +174,5 @@
     </inertial>
     <visual>
-      <origin xyz="0.1 0 -.10" rpy="0 0 0" />
+      <origin xyz="0.12 0 -.095" rpy="0 0 0" />
       <geometry>
         <mesh filename="file://$(find zbig_description)/meshes/narrowbot/collision-imu.stl" />
@@ -222,5 +217,5 @@
   </link>
   <joint name="laser_joint" type="fixed">
-    <origin xyz="-0.035 0.000 0.4" rpy="${lidar_roll} ${lidar_pitch} ${lidar_yaw}" />
+    <origin xyz="-0.030 0.000 0.4" rpy="${lidar_roll} ${lidar_pitch} ${lidar_yaw}" />
     <parent link="base_link" />
     <child link="laser_frame" />

Commit message: initial cbot load

File: src/zbig_description/urdf/bigbot_physical.urdf.xacro (robot description, xacro)
@@ -59,5 +59,5 @@
       <origin xyz="-0.0 0.0 0.0" rpy="1.57 0 0" />
       <geometry>
-        <mesh filename="file://$(find zbig_description)/meshes/narrowbot/collision-6inch-wheel.stl" />
+        <mesh filename="file://$(find zbig_description)/meshes/cbot/collision-6inch-wheel.stl" />
       </geometry>
       <material name="blue"/>
@@ -89,5 +89,5 @@
       <origin xyz="0 0.0 0" rpy="-1.57 0 0" />
       <geometry>
-        <mesh filename="file://$(find zbig_description)/meshes/narrowbot/collision-6inch-wheel.stl" />
+        <mesh filename="file://$(find zbig_description)/meshes/cbot/collision-6inch-wheel.stl" />
       </geometry>
       <material name="blue"/>
@@ -118,5 +118,5 @@
       <origin xyz="0 ${wheel_offset_z} 0" rpy="0 1.57 0" />
       <geometry>
-        <mesh filename="file://$(find zbig_description)/meshes/narrowbot/visual-caster-narrow1.stl" />
+        <mesh filename="file://$(find zbig_description)/meshes/cbot/visual-caster-narrow1.stl" />
       </geometry>
       <material name="silver"/>
@@ -147,5 +147,5 @@
       <origin xyz="0 ${wheel_offset_z} 0" rpy="0 -1.57 0.0" />
       <geometry>
-         <mesh filename="file://$(find zbig_description)/meshes/narrowbot/visual-caster-narrow1.stl" />
+         <mesh filename="file://$(find zbig_description)/meshes/cbot/visual-caster-narrow1.stl" />
       </geometry>
       <material name="silver"/>
@@ -176,5 +176,5 @@
       <origin xyz="0.12 0 -.095" rpy="0 0 0" />
       <geometry>
-        <mesh filename="file://$(find zbig_description)/meshes/narrowbot/collision-imu.stl" />
+        <mesh filename="file://$(find zbig_description)/meshes/cbot/collision-imu.stl" />
       </geometry>
       <material name="blue"/>
@@ -183,5 +183,5 @@
       <origin xyz="0.1 0 -.10" rpy="${imu_roll} ${imu_pitch} ${imu_yaw}" />
       <geometry>
-        <mesh filename="file://$(find zbig_description)/meshes/narrowbot/collision-imu.stl" />
+        <mesh filename="file://$(find zbig_description)/meshes/cbot/collision-imu.stl" />
       </geometry>
     </collision>
@@ -205,5 +205,5 @@
       <origin xyz="0 0 0" rpy="1.57 0 0" />
       <geometry>
-        <mesh filename="file://$(find zbig_description)/meshes/narrowbot/collision-lidar.stl" />
+        <mesh filename="file://$(find zbig_description)/meshes/cbot/collision-lidar.stl" />
       </geometry>
       <material name="black"/>
@@ -212,5 +212,5 @@
       <origin xyz="0 0 0" rpy="${lidar_roll} ${lidar_pitch} ${lidar_yaw}" />
       <geometry>
-        <mesh filename="file://$(find zbig_description)/meshes/narrowbot/collision-lidar.stl" />
+        <mesh filename="file://$(find zbig_description)/meshes/cbot/collision-lidar.stl" />
       </geometry>
     </collision>

File: src/zbig_description/urdf/cbot_chassis.urdf.xacro (robot description, xacro)
@@ -3,8 +3,8 @@
     <xacro:property name="wheel_radius" value="0.074"/>
     <xacro:property name="wheel_offset_y" value="0.15283"/>
-    <xacro:property name="wheel_offset_z" value="0.0225"/>
-    <xacro:property name="caster_wheel_radius" value="0.051"/>
+    <xacro:property name="wheel_offset_z" value="0.0"/>
+    <xacro:property name="caster_wheel_radius" value="0.0254"/>
     <xacro:property name="caster_wheel_offset_x" value="0.137"/>
-    <xacro:property name="caster_wheel_offset_y" value="0.095"/>
+    <xacro:property name="caster_wheel_offset_y" value="0.0"/>
     <xacro:property name="caster_wheel_offset_z" value="${wheel_offset_z - wheel_radius + caster_wheel_radius}"/>
     <xacro:property name="chassis_mass" value="10.0"/>
@@ -31,14 +31,14 @@
     <axis xyz="0 1 0" />
   </joint>
-  <joint name="caster_right_joint" type="fixed">
-    <origin xyz="${-caster_wheel_offset_x} ${-caster_wheel_offset_y} ${-caster_wheel_offset_z}" rpy="1.57 0 1.57" />
+  <joint name="caster_rear_joint" type="fixed">
+    <origin xyz="${-caster_wheel_offset_x} ${-caster_wheel_offset_y} ${caster_wheel_offset_z}" rpy="1.57 0 1.57" />
     <parent link="base_link" />
-    <child link="caster_right_link" />
+    <child link="caster_rear_link" />
     <axis xyz="0 0 0" />
   </joint>
-  <joint name="caster_left_joint" type="fixed">
-    <origin xyz="${-caster_wheel_offset_x} ${caster_wheel_offset_y} ${-caster_wheel_offset_z}" rpy="1.57 0 1.57" />
+  <joint name="caster_front_joint" type="fixed">
+    <origin xyz="${caster_wheel_offset_x} ${caster_wheel_offset_y} ${caster_wheel_offset_z}" rpy="1.57 0 1.57" />
     <parent link="base_link" />
-    <child link="caster_left_link" />
+    <child link="caster_front_link" />
     <axis xyz="0 0 0" />
   </joint>
@@ -56,5 +56,5 @@
       <origin xyz="0 0 0" rpy="0 0 0" />
       <geometry>
-        <mesh filename="file://$(find zbig_description)/meshes/narrowbot/collision-chassis-narrow1.stl" />
+        <mesh filename="file://$(find zbig_description)/meshes/cbot/collision-chassis-center1.stl" />
       </geometry>
       <material name="dark_grey"/>
@@ -63,5 +63,5 @@
       <origin xyz="0 0 0" rpy="0 0 0" />
       <geometry>
-        <mesh filename="file://$(find zbig_description)/meshes/narrowbot/collision-chassis-narrow1.stl" />
+        <mesh filename="file://$(find zbig_description)/meshes/cbot/collision-chassis-center1.stl" />
       </geometry>
     </collision>
@@ -79,5 +79,5 @@
       <origin xyz="-0.0 0.014 0.0" rpy="1.57 0 0" />
       <geometry>
-        <mesh filename="file://$(find zbig_description)/meshes/narrowbot/collision-6inch-wheel.stl" />
+        <mesh filename="file://$(find zbig_description)/meshes/cbot/collision-6inch-wheel.stl" />
       </geometry>
       <material name="blue"/>
@@ -103,5 +103,5 @@
       <origin xyz="0 -0.014 0" rpy="-1.57 0 0" />
       <geometry>
-        <mesh filename="file://$(find zbig_description)/meshes/narrowbot/collision-6inch-wheel.stl" />
+        <mesh filename="file://$(find zbig_description)/meshes/cbot/collision-6inch-wheel.stl" />
       </geometry>
       <material name="blue"/>
@@ -114,6 +114,6 @@
     </collision>
   </link>
-  <!-- RIGHT CASTER WHEEL LINK -->
-  <link name="caster_right_link">
+  <!-- REAR CASTER WHEEL LINK -->
+  <link name="caster_rear_link">
     <inertial>
       <origin xyz=".000112 -0.0155 -.00818" rpy="0 0 0" />
@@ -126,5 +126,5 @@
       <origin xyz="0 0 0" rpy="0 0 0" />
       <geometry>
-        <mesh filename="file://$(find zbig_description)/meshes/smallbot_caster_link.stl" />
+        <mesh filename="file://$(find zbig_description)/meshes/cbot/visual-caster-2inch.stl" />
       </geometry>
       <material name="silver"/>
@@ -133,10 +133,10 @@
       <origin xyz="0 0 0" rpy="0 0 0" />
       <geometry>
-        <sphere radius="${wheel_radius}"/>
+        <sphere radius="${caster_wheel_radius}"/>
       </geometry>
     </collision>
   </link>
-  <!-- LEFT CASTER WHEEL LINK -->
-  <link name="caster_left_link">
+  <!-- FRONT CASTER WHEEL LINK -->
+  <link name="caster_front_link">
     <inertial>
       <origin xyz=".000112 -0.0155 -.00818" rpy="0 0 0" />
@@ -149,5 +149,5 @@
       <origin xyz="0 0 0" rpy="0 0 0" />
       <geometry>
-        <mesh filename="file://$(find zbig_description)/meshes/smallbot_caster_link.stl" />
+        <mesh filename="file://$(find zbig_description)/meshes/cbot/visual-caster-2inch.stl" />
       </geometry>
       <material name="silver"/>
@@ -156,5 +156,5 @@
       <origin xyz="0 0 0" rpy="0 0 0" />
       <geometry>
-        <sphere radius="${wheel_radius}"/>
+        <sphere radius="${caster_wheel_radius}"/>
       </geometry>
     </collision>
@@ -180,5 +180,5 @@
   </gazebo>
   <!-- Caster Wheels -->
-  <gazebo reference="caster_right_link">
+  <gazebo reference="caster_rear_link">
     <mu1>0.1</mu1>
     <mu2>0.1</mu2>
@@ -188,5 +188,5 @@
     <maxVel>1.0</maxVel>
   </gazebo>
-  <gazebo reference="caster_left_link">
+  <gazebo reference="caster_front_link">
     <mu1>0.1</mu1>
     <mu2>0.1</mu2>

File: src/zbig_description/urdf/cbot_gazebo_control.xacro (robot description, xacro)
@@ -5,5 +5,5 @@
     <xacro:if value="$(arg is_sim)">
       <plugin name="gz_ros2_control::GazeboSimROS2ControlPlugin" filename="gz_ros2_control-system">
-        <parameters>$(find zbig_controller)/config/bigbot_controllers.yaml</parameters>
+        <parameters>$(find zbig_controller)/config/cbot_controllers.yaml</parameters>
       </plugin>
     </xacro:if>

File: src/zbig_description/urdf/imu_cbot.xacro (robot description, xacro)
@@ -6,5 +6,5 @@
   <!-- IMU JOINT -->
   <joint name="imu_joint" type="fixed">
-    <origin xyz="-0.04016 0.049755 0.064953" rpy="${imu_roll} ${imu_pitch} ${imu_yaw}" />
+    <origin xyz="0.151167 0.0 0.092" rpy="${imu_roll} ${imu_pitch} ${imu_yaw}" />
     <parent link="base_link" />
     <child link="imu_link" />
@@ -21,14 +21,14 @@
     </inertial>
     <visual>
-      <origin xyz="0 0 0" rpy="0 0 0" />
+      <origin xyz="0.125 0 -0.093625" rpy="0 0 0" />
       <geometry>
-        <mesh filename="file://$(find zbig_description)/meshes/narrowbot/collision-imu.stl" />
+        <mesh filename="file://$(find zbig_description)/meshes/cbot/collision-imu.stl" />
       </geometry>
       <material name="blue"/>
     </visual>
     <collision>
-      <origin xyz="0 0 0" rpy="${imu_roll} ${imu_pitch} ${imu_yaw}" />
+      <origin xyz="0.125 0 -0.093625" rpy="${imu_roll} ${imu_pitch} ${imu_yaw}" />
       <geometry>
-        <mesh filename="file://$(find zbig_description)/meshes/narrowbot/collision-imu.stl" />
+        <mesh filename="file://$(find zbig_description)/meshes/cbot/collision-imu.stl" />
       </geometry>
     </collision>

File: src/zbig_description/urdf/lidar_cbot.xacro (robot description, xacro)
@@ -6,5 +6,5 @@
   <!-- LIDAR JOINT -->
   <joint name="laser_joint" type="fixed">
-    <origin xyz="-0.013456 0.000513 0.140452" rpy="${lidar_roll} ${lidar_pitch} ${lidar_yaw}" />
+    <origin xyz="0.151167 0.000513 0.140452" rpy="${lidar_roll} ${lidar_pitch} ${lidar_yaw}" />
     <parent link="base_link" />
     <child link="laser_frame" />
@@ -23,5 +23,5 @@
       <origin xyz="0 0 0" rpy="1.57 0 3.14" />
       <geometry>
-        <mesh filename="file://$(find zbig_description)/meshes/narrowbot/collision-lidar.stl" />
+        <mesh filename="file://$(find zbig_description)/meshes/cbot/collision-lidar.stl" />
       </geometry>
       <material name="black"/>
@@ -30,5 +30,5 @@
       <origin xyz="0 0 0" rpy="${lidar_roll} ${lidar_pitch} ${lidar_yaw}" />
       <geometry>
-        <mesh filename="file://$(find zbig_description)/meshes/narrowbot/collision-lidar.stl" />
+        <mesh filename="file://$(find zbig_description)/meshes/cbot/collision-lidar.stl" />
       </geometry>
     </collision>
@@ -47,11 +47,11 @@
             <samples>360</samples>
             <resolution>1.00000</resolution>
-            <min_angle>-2.2</min_angle>
-            <max_angle>2.2</max_angle>
+            <min_angle>-1.57</min_angle>
+            <max_angle>1.57</max_angle>
           </horizontal>
         </scan>
         <range>
           <min>0.120000</min>
-          <max>12.0</max>
+          <max>10.0</max>
           <resolution>0.02</resolution>
         </range>
