Commit message: added use_depth_cam arg

File: src/zbig_description/urdf/smallbot.urdf.xacro (robot description, xacro)
@@ -19,4 +19,4 @@
   <!-- Include sensors -->
   <xacro:include filename="$(find zbig_description)/urdf/camera_cbot.xacro" />
-  <xacro:include filename="$(find zbig_description)/urdf/depth_camera_cbot.xacro" />
+  <!-- <xacro:include filename="$(find zbig_description)/urdf/depth_camera_cbot.xacro" /> -->
 </robot>

File: src/zbig_description/urdf/smallbot_physical.urdf.xacro (robot description, xacro)
@@ -3,5 +3,5 @@
     <xacro:property name="robot_pitch" value="-0.02618"/>
     <xacro:property name="wheel_radius" value="0.0335"/>
-    <xacro:property name="wheel_offset_y" value="0.160"/>
+    <xacro:property name="wheel_offset_y" value="0.140"/>
     <xacro:property name="wheel_offset_z" value="0.0"/>
     <xacro:property name="caster_wheel_radius" value="0.0335"/>
