Commit message: smallbot calibrated

File: src/zbig_description/urdf/smallbot_physical.urdf.xacro (robot description, xacro)
@@ -3,5 +3,5 @@
     <xacro:property name="robot_pitch" value="-0.02618"/>
     <xacro:property name="wheel_radius" value="0.0335"/>
-    <xacro:property name="wheel_offset_y" value="0.140"/>
+    <xacro:property name="wheel_offset_y" value="0.16"/>
     <xacro:property name="wheel_offset_z" value="0.0"/>
     <xacro:property name="caster_wheel_radius" value="0.0335"/>

Commit message: more smallbot tuning

File: src/zbig_description/urdf/smallbot_physical.urdf.xacro (robot description, xacro)
@@ -3,5 +3,5 @@
     <xacro:property name="robot_pitch" value="-0.02618"/>
     <xacro:property name="wheel_radius" value="0.0335"/>
-    <xacro:property name="wheel_offset_y" value="0.16"/>
+    <xacro:property name="wheel_offset_y" value="0.144"/>
     <xacro:property name="wheel_offset_z" value="0.0"/>
     <xacro:property name="caster_wheel_radius" value="0.0335"/>
