Commit message: real bigbot is now cbot

File: src/zbig_description/urdf/camera_cbot.xacro (robot description, xacro)
@@ -4,5 +4,5 @@
         <parent link="base_link"/>
         <child link="camera_link"/>
-        <origin xyz="0.08 0.17 0.30" rpy="0 0.09 0"/>
+        <origin xyz="0.190338 0.0 0.108" rpy="0 0.0 0"/>
     </joint>
     <link name="camera_link">

File: src/zbig_description/urdf/cbot_chassis.urdf.xacro (robot description, xacro)
@@ -56,5 +56,5 @@
       <origin xyz="0 0 0" rpy="0 0 0" />
       <geometry>
-        <mesh filename="file://$(find zbig_description)/meshes/cbot/collision-chassis-center1.stl" />
+        <mesh filename="file://$(find zbig_description)/meshes/cbot/collision-chassis-center_short.stl" />
       </geometry>
       <material name="dark_grey"/>
@@ -63,5 +63,5 @@
       <origin xyz="0 0 0" rpy="0 0 0" />
       <geometry>
-        <mesh filename="file://$(find zbig_description)/meshes/cbot/collision-chassis-center1.stl" />
+        <mesh filename="file://$(find zbig_description)/meshes/cbot/collision-chassis-center_short.stl" />
       </geometry>
     </collision>

File: src/zbig_description/urdf/depth_camera_cbot.xacro (robot description, xacro)
@@ -5,5 +5,5 @@
         <parent link="base_link"/>
         <child link="depth_camera_link"/>
-        <origin xyz="0.08 0.0 0.050" rpy="0 0 0"/>
+        <origin xyz="0.190338 0.0 0.108" rpy="0 0 0"/>
     </joint>
         <joint name="depth_camera_optical_joint" type="fixed">

File: src/zbig_description/urdf/imu_cbot.xacro (robot description, xacro)
@@ -6,5 +6,5 @@
   <!-- IMU JOINT -->
   <joint name="imu_joint" type="fixed">
-    <origin xyz="0.151167 0.0 0.092" rpy="${imu_roll} ${imu_pitch} ${imu_yaw}" />
+    <origin xyz="0.0 0.1715 0.104" rpy="${imu_roll} ${imu_pitch} ${imu_yaw}" />
     <parent link="base_link" />
     <child link="imu_link" />

File: src/zbig_description/urdf/lidar_cbot.xacro (robot description, xacro)
@@ -6,5 +6,5 @@
   <!-- LIDAR JOINT -->
   <joint name="laser_joint" type="fixed">
-    <origin xyz="0.151167 0.000513 0.140452" rpy="${lidar_roll} ${lidar_pitch} ${lidar_yaw}" />
+    <origin xyz="0.127768 0.00 0.216947" rpy="${lidar_roll} ${lidar_pitch} ${lidar_yaw}" />
     <parent link="base_link" />
     <child link="laser_frame" />
