Commit message: added gazebo to depth cam urdf

File: src/zbig_description/urdf/depthai_descr.urdf.xacro (robot description, xacro)
@@ -104,3 +104,48 @@
 		</joint>
 	</xacro:if>
+	<!-- GAZEBO STUFF -->
+    <gazebo reference="depth_camera_link">
+        <material>Gazebo/Red</material>
+      <sensor name="depth_camera" type="depth_camera">
+        <always_on>true</always_on>
+        <visualize>true</visualize>
+        <update_rate>5.0</update_rate>
+        <topic>depth_camera</topic>
+        <gz_frame_id>depth_camera_link</gz_frame_id>
+        <camera name="OAK">
+          <camera_info_topic>depth_camera_info</camera_info_topic>
+          <horizontal_fov>1.20428</horizontal_fov>
+          <!-- <vertical_fov>0.05</vertical_fov>  -->
+          <image>
+            <width>480</width>
+            <height>480</height>
+          </image>
+          <clip>
+            <near>0.05</near>
+            <far>3</far>
+          </clip>
+          <depth_camera>
+            <output>depths</output>
+            <clip>
+              <near>0.05</near>
+              <far>4</far>
+            </clip>
+          </depth_camera>
+          <optical_frame_id>depth_camera_link</optical_frame_id>
+        </camera>
+        <baseline>0.2</baseline>
+        <pointCloudCutoff>0.5</pointCloudCutoff>
+        <pointCloudCutoffMax>3.0</pointCloudCutoffMax>
+        <distortionK1>0</distortionK1>
+        <distortionK2>0</distortionK2>
+        <distortionK3>0</distortionK3>
+        <distortionT1>0</distortionT1>
+        <distortionT2>0</distortionT2>
+        <CxPrime>0</CxPrime>
+        <Cx>0</Cx>
+        <Cy>0</Cy>
+        <focalLength>0</focalLength>
+        <hackBaseline>0</hackBaseline>
+      </sensor>
+    </gazebo>
 </robot>
